Commit message: Added option to insert simple wheels on feet

File: urdf/leg.xacro (robot description, xacro)
@@ -2,5 +2,5 @@
     <xacro:include filename="$(find mulinex_description)/urdf/links.xacro" />
     <xacro:property name="PI" value="3.141592" />
-    <xacro:macro name="leg" params="prefix gazebo jnt_pref simplify_meshes">
+    <xacro:macro name="leg" params="prefix gazebo jnt_pref simplify_meshes wheels">
         <!-- Module 1 -->
         <xacro:hip
@@ -19,5 +19,6 @@
             gazebo="${gazebo}"
             jnt_pref="${jnt_pref}"
-            simplify_meshes="${simplify_meshes}" />
+            simplify_meshes="${simplify_meshes}"
+            wheels="${wheels}" />
     </xacro:macro>
 </robot>

File: urdf/links.xacro (robot description, xacro)
@@ -335,5 +335,5 @@
     </xacro:macro>
     <!-- LOWER LEG -->
-    <xacro:macro name="lower_leg" params="prefix gazebo jnt_pref simplify_meshes">
+    <xacro:macro name="lower_leg" params="prefix gazebo jnt_pref simplify_meshes wheels">
         <!-- Transformation based on the position of each link -->
         <xacro:if value="${prefix == 'LF'}">
@@ -413,5 +413,5 @@
                         <origin xyz="0 0 0" rpy="0 ${-PI/2} 0" />
                         <geometry>
-                            <mesh filename="${mulinex_lower_leg_right}" />
+                            <mesh filename="${msphereulinex_lower_leg_right}" />
                         </geometry>
                     </xacro:if>
@@ -511,61 +511,162 @@
             </gazebo>
         </xacro:if>
-        <joint name="${prefix}_ANKLE" type="fixed">
-            <parent link="${prefix}_LOWER_LEG" />
-            <child link="${prefix}_FOOT" />
-            <xacro:if value="${prefix == 'LF'}">
-                <origin xyz="${KFE_2_FOOT_x} ${KFE_2_FOOT_y} 0" rpy="0 0 0" />
+        <!-- Include wheels -->
+        <xacro:if value="${wheels}">
+            <joint name="${prefix}_ANKLE" type="continuous">
+                <parent link="${prefix}_LOWER_LEG" />
+                <child link="${prefix}_WHEEL" />
+                <xacro:if value="${prefix == 'LF'}">
+                    <origin xyz="${KFE_2_FOOT_x} ${KFE_2_FOOT_y} 0" rpy="0 0 0" />
+                    <axis xyz="0 1 0" />
+                </xacro:if>
+                <xacro:if value="${prefix == 'LH'}">
+                    <origin xyz="${-KFE_2_FOOT_x} ${KFE_2_FOOT_y} 0" rpy="0 0 0" />
+                    <axis xyz="0 1 0" />
+                </xacro:if>
+                <xacro:if value="${prefix == 'RF'}">
+                    <origin xyz="${KFE_2_FOOT_x} ${-KFE_2_FOOT_y} 0" rpy="0 0 0" />
+                    <axis xyz="0 1 0" />
+                </xacro:if>
+                <xacro:if value="${prefix == 'RH'}">
+                    <origin xyz="${-KFE_2_FOOT_x} ${-KFE_2_FOOT_y} 0" rpy="0 0 0" />
+                    <axis xyz="0 1 0" />
+                </xacro:if>
+            </joint>
+            <link name="${prefix}_WHEEL">
+                <visual>
+                    <material name="white" />
+                    <origin xyz="0 0 0" rpy="${PI/2} 0 0" />
+                    <geometry>
+                        <cylinder length="0.10" radius="0.015" />
+                    </geometry>
+                </visual>
+                <xacro:if value="${simplify_meshes}">
+                    <collision>
+                        <origin xyz="0 0 0" rpy="${PI/2} 0 0" />
+                        <geometry>
+                            <cylinder length="0.10" radius="0.015" />
+                        </geometry>
+                    </collision>
+                </xacro:if>
+            </link>
+            <xacro:if value="${gazebo}">
+                <gazebo reference="${prefix}_WHEEL">
+                    <material>Gazebo/White</material>
+                    <collision>
+                        <surface>
+                            <friction>
+                                <ode>
+                                    <mu>0.6</mu>
+                                    <mu2>0.6</mu2>
+                                    <slip1>0</slip1>
+                                    <slip2>0</slip2>
+                                </ode>
+                            </friction>
+                            <contact>
+                                <ode>
+                                    <kp>10000.0</kp>
+                                    <kd>100.0</kd>
+                                    <min_depth>0.001</min_depth>
+                                </ode>
+                            </contact>
+                        </surface>
+                    </collision>
+                    <sensor name="${prefix}_contactsensor_sensor" type="contact">
+                        <always_on>true</always_on>
+                        <update_rate>50</update_rate>
+                        <contact>
+                            <collision>
+                                ${prefix}_LOWER_LEG_fixed_joint_lump__${prefix}_FOOT_collision_1</collision>
+                        </contact>
+                    </sensor>
+                </gazebo>
             </xacro:if>
-            <xacro:if value="${prefix == 'LH'}">
-                <origin xyz="${-KFE_2_FOOT_x} ${KFE_2_FOOT_y} 0" rpy="0 0 0" />
+            <joint name="${prefix}_DIRECTION" type="fixed">
+                <parent link="${prefix}_WHEEL" />
+                <child link="${prefix}_INDICATOR" />
+                <xacro:if value="${prefix == 'LF'}">
+                    <origin xyz="0 0.0501 0" rpy="0 0 0" />
+                </xacro:if>
+                <xacro:if value="${prefix == 'LH'}">
+                    <origin xyz="0 0.0501 0" rpy="0 0 0" />
+                </xacro:if>
+                <xacro:if value="${prefix == 'RF'}">
+                    <origin xyz="0 -0.0501 0" rpy="0 0 0" />
+                </xacro:if>
+                <xacro:if value="${prefix == 'RH'}">
+                    <origin xyz="0 -0.0501 0" rpy="0 0 0" />
+                </xacro:if>
+            </joint>
+            <link name="${prefix}_INDICATOR">
+                <visual>
+                    <origin xyz="0 0 0.0075" rpy="0 0 0" />
+                    <geometry>
+                        <box size="0.004 0.0001 0.015" />
+                    </geometry>
+                    <material name="red" />
+                </visual>
+            </link>
+        </xacro:if>
+        <!-- Without wheels -->
+        <xacro:unless value="${wheels}">
+            <joint name="${prefix}_ANKLE" type="fixed">
+                <parent link="${prefix}_LOWER_LEG" />
+                <child link="${prefix}_FOOT" />
+                <xacro:if value="${prefix == 'LF'}">
+                    <origin xyz="${KFE_2_FOOT_x} ${KFE_2_FOOT_y} 0" rpy="0 0 0" />
+                </xacro:if>
+                <xacro:if value="${prefix == 'LH'}">
+                    <origin xyz="${-KFE_2_FOOT_x} ${KFE_2_FOOT_y} 0" rpy="0 0 0" />
+                </xacro:if>
+                <xacro:if value="${prefix == 'RF'}">
+                    <origin xyz="${KFE_2_FOOT_x} ${-KFE_2_FOOT_y} 0" rpy="0 0 0" />
+                </xacro:if>
+                <xacro:if value="${prefix == 'RH'}">
+                    <origin xyz="${-KFE_2_FOOT_x} ${-KFE_2_FOOT_y} 0" rpy="0 0 0" />
+                </xacro:if>
+            </joint>
+            <link name="${prefix}_FOOT">
+                <xacro:if value="${simplify_meshes}">
+                    <collision>
+                        <origin xyz="0 0 0" rpy="0 0 0" />
+                        <geometry>
+                            <sphere radius="0.015" />
+                        </geometry>
+                    </collision>
+                </xacro:if>
+            </link>
+            <xacro:if value="${gazebo}">
+                <gazebo reference="${prefix}_FOOT">
+                    <material>Gazebo/White</material>
+                    <collision>
+                        <surface>
+                            <friction>
+                                <ode>
+                                    <mu>0.6</mu>
+                                    <mu2>0.6</mu2>
+                                    <slip1>0</slip1>
+                                    <slip2>0</slip2>
+                                </ode>
+                            </friction>
+                            <contact>
+                                <ode>
+                                    <kp>10000.0</kp>
+                                    <kd>100.0</kd>
+                                    <min_depth>0.001</min_depth>
+                                </ode>
+                            </contact>
+                        </surface>
+                    </collision>
+                    <sensor name="${prefix}_contactsensor_sensor" type="contact">
+                        <always_on>true</always_on>
+                        <update_rate>50</update_rate>
+                        <contact>
+                            <collision>
+                                ${prefix}_LOWER_LEG_fixed_joint_lump__${prefix}_FOOT_collision_1</collision>
+                        </contact>
+                    </sensor>
+                </gazebo>
             </xacro:if>
-            <xacro:if value="${prefix == 'RF'}">
-                <origin xyz="${KFE_2_FOOT_x} ${-KFE_2_FOOT_y} 0" rpy="0 0 0" />
-            </xacro:if>
-            <xacro:if value="${prefix == 'RH'}">
-                <origin xyz="${-KFE_2_FOOT_x} ${-KFE_2_FOOT_y} 0" rpy="0 0 0" />
-            </xacro:if>
-        </joint>
-        <link name="${prefix}_FOOT">
-            <xacro:if value="${simplify_meshes}">
-                <collision>
-                    <origin xyz="0 0 0" rpy="0 0 0" />
-                    <geometry>
-                        <sphere radius="0.015" />
-                    </geometry>
-                </collision>
-            </xacro:if>
-        </link>
-        <xacro:if value="${gazebo}">
-            <gazebo reference="${prefix}_FOOT">
-                <material>Gazebo/White</material>
-                <collision>
-                    <surface>
-                        <friction>
-                            <ode>
-                                <mu>0.6</mu>
-                                <mu2>0.6</mu2>
-                                <slip1>0</slip1>
-                                <slip2>0</slip2>
-                            </ode>
-                        </friction>
-                        <contact>
-                            <ode>
-                                <kp>10000.0</kp>
-                                <kd>100.0</kd>
-                                <min_depth>0.001</min_depth>
-                            </ode>
-                        </contact>
-                    </surface>
-                </collision>
-                <sensor name="${prefix}_contactsensor_sensor" type="contact">
-                    <always_on>true</always_on>
-                    <update_rate>50</update_rate>
-                    <contact>
-                        <collision>${prefix}_LOWER_LEG_fixed_joint_lump__${prefix}_FOOT_collision_1</collision>
-                    </contact>
-                </sensor>
-            </gazebo>
-        </xacro:if>
+        </xacro:unless>
     </xacro:macro>
 </robot>

File: urdf/mulinex.xacro (robot description, xacro)
@@ -6,4 +6,5 @@
     <xacro:property name="use_gazebo" value="true" />
     <xacro:property name="simplify_meshes_lower_leg" value="true"/>
+    <xacro:property name="add_wheels" value="false"/>
     <xacro:property name="jnt_prefix" value="" />
     <xacro:property name="hind_haa" value="0.0" />
@@ -40,20 +41,24 @@
         gazebo="${use_gazebo}"
         jnt_pref="${jnt_prefix}"
-        simplify_meshes="${simplify_meshes_lower_leg}" />
+        simplify_meshes="${simplify_meshes_lower_leg}"
+        wheels="${add_wheels}" />
     <xacro:leg
         prefix="LF"
         gazebo="${use_gazebo}"
         jnt_pref="${jnt_prefix}"
-        simplify_meshes="${simplify_meshes_lower_leg}" />
+        simplify_meshes="${simplify_meshes_lower_leg}"
+        wheels="${add_wheels}" />
     <xacro:leg
         prefix="RF"
         gazebo="${use_gazebo}"
         jnt_pref="${jnt_prefix}"
-        simplify_meshes="${simplify_meshes_lower_leg}" />
+        simplify_meshes="${simplify_meshes_lower_leg}"
+        wheels="${add_wheels}" />
     <xacro:leg
         prefix="RH"
         gazebo="${use_gazebo}"
         jnt_pref="${jnt_prefix}"
-        simplify_meshes="${simplify_meshes_lower_leg}" />
+        simplify_meshes="${simplify_meshes_lower_leg}"
+        wheels="${add_wheels}" />
     <xacro:if value="${use_gazebo}">
         <gazebo reference="base_link">
