Commit message: Adjusted joint axis

File: urdf/links.xacro (robot description, xacro)
@@ -184,4 +184,5 @@
             <xacro:property name="hip_to_upper_leg_xyz" value="${HAA_2_HFE_x} ${HAA_2_HFE_y} 0" />
             <xacro:property name="hip_to_upper_leg_rpy" value="0 0 0" />
+            <xacro:property name="axis" value="0 1 0"/>
         </xacro:if>
         <xacro:if
@@ -189,4 +190,5 @@
             <xacro:property name="hip_to_upper_leg_xyz" value="${-HAA_2_HFE_x} ${HAA_2_HFE_y} 0" />
             <xacro:property name="hip_to_upper_leg_rpy" value="0 0 0" />
+            <xacro:property name="axis" value="0 1 0" />
         </xacro:if>
         <xacro:if
@@ -194,4 +196,5 @@
             <xacro:property name="hip_to_upper_leg_xyz" value="${HAA_2_HFE_x} ${-HAA_2_HFE_y} 0" />
             <xacro:property name="hip_to_upper_leg_rpy" value="0 0 0" />
+            <xacro:property name="axis" value="0 -1 0" />
         </xacro:if>
         <xacro:if
@@ -199,4 +202,5 @@
             <xacro:property name="hip_to_upper_leg_xyz" value="${-HAA_2_HFE_x} ${-HAA_2_HFE_y} 0" />
             <xacro:property name="hip_to_upper_leg_rpy" value="0 0 0" />
+            <xacro:property name="axis" value="0 -1 0" />
         </xacro:if>
         <xacro:property name="upper_to_lower_leg_rpy" value="0 0 0" />
@@ -206,5 +210,5 @@
             <child link="${jnt_pref}${prefix}_UPPER_LEG" />
             <origin xyz="${hip_to_upper_leg_xyz}" rpy="${hip_to_upper_leg_rpy}" />
-            <axis xyz="0 -1 0" />
+            <axis xyz="${axis}" />
             <limit effort="2.7" lower="-${PI}" upper="${PI}" velocity="1000" />
             <!-- <dynamics damping="0.7" friction="100.0" /> -->
@@ -335,16 +339,20 @@
         <xacro:if value="${prefix == 'LF'}">
             <xacro:property name="upper_to_lower_leg_xyz" value="${HFE_2_KFE_x} ${HFE_2_KFE_y} 0" />
+            <xacro:property name="axis" value="0 1 0" />
         </xacro:if>
         <xacro:if
             value="${prefix == 'LH'}">
             <xacro:property name="upper_to_lower_leg_xyz" value="${-HFE_2_KFE_x} ${HFE_2_KFE_y} 0" />
+            <xacro:property name="axis" value="0 1 0" />
         </xacro:if>
         <xacro:if
             value="${prefix == 'RF'}">
             <xacro:property name="upper_to_lower_leg_xyz" value="${HFE_2_KFE_x} ${-HFE_2_KFE_y} 0" />
+            <xacro:property name="axis" value="0 -1 0" />
         </xacro:if>
         <xacro:if
             value="${prefix == 'RH'}">
             <xacro:property name="upper_to_lower_leg_xyz" value="${-HFE_2_KFE_x} ${-HFE_2_KFE_y} 0" />
+            <xacro:property name="axis" value="0 -1 0" />
         </xacro:if>
         <xacro:property name="upper_to_lower_leg_rpy" value="0 0 0" />
@@ -354,5 +362,5 @@
             <child link="${jnt_pref}${prefix}_LOWER_LEG" />
             <origin xyz="${upper_to_lower_leg_xyz}" rpy="${upper_to_lower_leg_rpy}" />
-            <axis xyz="0 -1 0" />
+            <axis xyz="${axis}" />
             <limit effort="2.7" lower="-${PI}" upper="${PI}" velocity="1000" />
             <!-- <dynamics damping="0.7" friction="100.0" /> -->

Commit message: update xacro, fix error

File: urdf/links.xacro (robot description, xacro)
@@ -239,5 +239,5 @@
                     <origin xyz="0 0 0" rpy="0 0 0" />
                     <geometry>
-                        <mesh filename="${mulinex_module_right_hind}" />
+                        <mesh filename="${mulinex_module_right_hind}"/>
                     </geometry>
                 </xacro:if>

File: urdf/mulinex.xacro (robot description, xacro)
@@ -196,57 +196,58 @@
         </ros2_control>
         <gazebo reference="base_link">
-    <sensor name="br_imu" type="imu">
-        <always_on>true</always_on>
-        <update_rate>100</update_rate>
-        <imu>
-          <angular_velocity>
-            <x>
-              <noise type="gaussian">
-                <mean>0.0</mean>
-                <stddev>2e-4</stddev>
-              </noise>
-            </x>
-            <y>
-              <noise type="gaussian">
-                <mean>0.0</mean>
-                <stddev>2e-4</stddev>
-              </noise>
-            </y>
-            <z>
-              <noise type="gaussian">
-                <mean>0.0</mean>
-                <stddev>2e-4</stddev>
-              </noise>
-            </z>
-          </angular_velocity>
-          <linear_acceleration>
-            <x>
-              <noise type="gaussian">
-                <mean>0.0</mean>
-                <stddev>1.7e-2</stddev>
-              </noise>
-            </x>
-            <y>
-              <noise type="gaussian">
-                <mean>0.0</mean>
-                <stddev>1.7e-2</stddev>
-              </noise>
-            </y>
-            <z>
-              <noise type="gaussian">
-                <mean>0.0</mean>
-                <stddev>1.7e-2</stddev>
-              </noise>
-            </z>
-          </linear_acceleration>
-        </imu>
-        <plugin name="bytes_imu" filename="libgazebo_ros_imu_sensor.so">
-            <ros>
-                <namespace>imu</namespace>
-                <remapping>~/out:=data</remapping>
-            </ros>
-            <initial_orientation_as_reference>false</initial_orientation_as_reference>
-        </plugin>
-    </sensor>
+            <sensor name="br_imu" type="imu">
+                <always_on>true</always_on>
+                <update_rate>100</update_rate>
+                <imu>
+                <angular_velocity>
+                    <x>
+                    <noise type="gaussian">
+                        <mean>0.0</mean>
+                        <stddev>2e-4</stddev>
+                    </noise>
+                    </x>
+                    <y>
+                    <noise type="gaussian">
+                        <mean>0.0</mean>
+                        <stddev>2e-4</stddev>
+                    </noise>
+                    </y>
+                    <z>
+                    <noise type="gaussian">
+                        <mean>0.0</mean>
+                        <stddev>2e-4</stddev>
+                    </noise>
+                    </z>
+                </angular_velocity>
+                <linear_acceleration>
+                    <x>
+                    <noise type="gaussian">
+                        <mean>0.0</mean>
+                        <stddev>1.7e-2</stddev>
+                    </noise>
+                    </x>
+                    <y>
+                    <noise type="gaussian">
+                        <mean>0.0</mean>
+                        <stddev>1.7e-2</stddev>
+                    </noise>
+                    </y>
+                    <z>
+                    <noise type="gaussian">
+                        <mean>0.0</mean>
+                        <stddev>1.7e-2</stddev>
+                    </noise>
+                    </z>
+                </linear_acceleration>
+                </imu>
+                <plugin name="bytes_imu" filename="libgazebo_ros_imu_sensor.so">
+                    <ros>
+                        <namespace>imu</namespace>
+                        <remapping>~/out:=data</remapping>
+                    </ros>
+                    <initial_orientation_as_reference>false</initial_orientation_as_reference>
+                </plugin>
+            </sensor>
+        </gazebo>
     </xacro:if>
     <xacro:unless value="${use_gazebo}">

Commit message: Changed maximum motor torques from 5 to 10 N/m

File: urdf/links.xacro (robot description, xacro)
@@ -211,5 +211,5 @@
             <origin xyz="${hip_to_upper_leg_xyz}" rpy="${hip_to_upper_leg_rpy}" />
             <axis xyz="${axis}" />
-            <limit effort="5.0" lower="-${PI}" upper="${PI}" velocity="1000" />
+            <limit effort="10.0" lower="-${2*PI}" upper="${2*PI}" velocity="1000" />
             <!-- <dynamics damping="0.7" friction="100.0" /> -->
         </joint>
@@ -363,5 +363,5 @@
             <origin xyz="${upper_to_lower_leg_xyz}" rpy="${upper_to_lower_leg_rpy}" />
             <axis xyz="${axis}" />
-            <limit effort="5.0" lower="-${PI}" upper="${PI}" velocity="1000" />
+            <limit effort="10.0" lower="-${2*PI}" upper="${2*PI}" velocity="1000" />
             <!-- <dynamics damping="0.7" friction="100.0" /> -->
         </joint>
